Commit message: Mixed iiwa_gazebo and iiwa_description in one folder, some commits ago modelname changed from mw_iiwa to iiwa, which restored the color of the robot

File: src/iiwa_gazebo/urdf/iiwa14.urdf (robot description, URDF)
Before this commit: robot iiwa14, 11 links, 10 joints
Links:
- link iiwa_link_0: geometry collision mesh filename=package://iiwa_gazebo/meshes/iiwa14/collision/link_0.stl; visual mesh filename=package://iiwa_gazebo/meshes/iiwa14/visual/link_0.stl
- link iiwa_link_1: geometry collision mesh filename=package://iiwa_gazebo/meshes/iiwa14/collision/link_1.stl; visual mesh filename=package://iiwa_gazebo/meshes/iiwa14/visual/link_1.stl
- link iiwa_link_2: geometry collision mesh filename=package://iiwa_gazebo/meshes/iiwa14/collision/link_2.stl; visual mesh filename=package://iiwa_gazebo/meshes/iiwa14/visual/link_2.stl
- link iiwa_link_3: geometry collision mesh filename=package://iiwa_gazebo/meshes/iiwa14/collision/link_3.stl; visual mesh filename=package://iiwa_gazebo/meshes/iiwa14/visual/link_3.stl
- link iiwa_link_4: geometry collision mesh filename=package://iiwa_gazebo/meshes/iiwa14/collision/link_4.stl; visual mesh filename=package://iiwa_gazebo/meshes/iiwa14/visual/link_4.stl
- link iiwa_link_5: geometry collision mesh filename=package://iiwa_gazebo/meshes/iiwa14/collision/link_5.stl; visual mesh filename=package://iiwa_gazebo/meshes/iiwa14/visual/link_5.stl
- link iiwa_link_6: geometry collision mesh filename=package://iiwa_gazebo/meshes/iiwa14/collision/link_6.stl; visual mesh filename=package://iiwa_gazebo/meshes/iiwa14/visual/link_6.stl
- link iiwa_link_7: geometry collision mesh filename=package://iiwa_gazebo/meshes/iiwa14/collision/link_7.stl; visual mesh filename=package://iiwa_gazebo/meshes/iiwa14/visual/link_7.stl

File: src/iiwa_gazebo/urdf/iiwa14.urdf.xacro (robot description, xacro)
@@ -1,7 +1,7 @@
 <robot name="iiwa14" xmlns:xacro="http://www.ros.org/wiki/xacro">
   <!-- Import Rviz colors -->
-  <xacro:include filename="$(find iiwa_description)/urdf/materials.xacro" />
+  <xacro:include filename="$(find iiwa_gazebo)/urdf/materials.xacro" />
   <!--Import the lbr iiwa macro -->
-  <xacro:include filename="$(find iiwa_description)/urdf/iiwa14.xacro"/>
+  <xacro:include filename="$(find iiwa_gazebo)/urdf/iiwa14.xacro"/>
   <xacro:arg name="robot_name" default="iiwa"/>
   <!-- Fix to world just for testing -->
@@ -9,5 +9,5 @@
   <!--iiwa-->
   <xacro:iiwa14 robot_name="$(arg robot_name)" parent="world">
-    <origin xyz="0 0 0.0" rpy="0 0 0" />
+    <origin xyz="0 0 0.0" rpy="0 0 0"/>
   </xacro:iiwa14>
 </robot>

File: src/iiwa_gazebo/urdf/iiwa14.xacro (robot description, xacro)
@@ -1,7 +1,7 @@
 <robot xmlns:xacro="http://www.ros.org/wiki/xacro">
   <!-- Import all Gazebo-customization elements, including Gazebo colors -->
-  <xacro:include filename="$(find iiwa_description)/urdf/iiwa.gazebo.xacro" />
+  <xacro:include filename="$(find iiwa_gazebo)/urdf/iiwa.gazebo.xacro" />
   <!-- Include Utilities -->
-  <xacro:include filename="$(find iiwa_description)/urdf/utilities.xacro" />
+  <xacro:include filename="$(find iiwa_gazebo)/urdf/utilities.xacro" />
   <!-- some constants -->
   <xacro:property name="safety_controller_k_pos" value="100" />
@@ -13,5 +13,5 @@
     <!--joint between {parent} and link_0-->
     <joint name="${parent}_${robot_name}_joint" type="fixed">
-      <insert_block name="origin"/>
+      <xacro:insert_block name="origin"/>
       <parent link="${parent}"/>
       <child link="${robot_name}_link_0"/>
@@ -26,5 +26,5 @@
         <origin xyz="0 0 0" rpy="0 0 0"/>
         <geometry>
-          <mesh filename="package://iiwa_description/meshes/iiwa14/visual/link_0.stl"/>
+          <mesh filename="package://iiwa_gazebo/meshes/iiwa14/visual/link_0.stl"/>
         </geometry>
         <material name="Grey"/>
@@ -33,5 +33,5 @@
         <origin xyz="0 0 0" rpy="0 0 0"/>
         <geometry>
-          <mesh filename="package://iiwa_description/meshes/iiwa14/collision/link_0.stl"/>
+          <mesh filename="package://iiwa_gazebo/meshes/iiwa14/collision/link_0.stl"/>
         </geometry>
         <material name="Grey"/>
@@ -67,12 +67,12 @@
         <origin xyz="0 0 0" rpy="0 0 0"/>
         <geometry>
-          <mesh filename="package://iiwa_description/meshes/iiwa14/visual/link_1.stl"/>
-        </geometry>
-        <material name="Orange"/>
-      </visual>
-      <collision>
-        <origin xyz="0 0 0" rpy="0 0 0"/>
-        <geometry>
-          <mesh filename="package://iiwa_description/meshes/iiwa14/collision/link_1.stl"/>
+          <mesh filename="package://iiwa_gazebo/meshes/iiwa14/visual/link_1.stl"/>
+        </geometry>
+        <material name="Orange"/>
+      </visual>
+      <collision>
+        <origin xyz="0 0 0" rpy="0 0 0"/>
+        <geometry>
+          <mesh filename="package://iiwa_gazebo/meshes/iiwa14/collision/link_1.stl"/>
         </geometry>
         <material name="Orange"/>
@@ -102,12 +102,12 @@
         <origin xyz="0 0 0" rpy="0 0 0"/>
         <geometry>
-          <mesh filename="package://iiwa_description/meshes/iiwa14/visual/link_2.stl"/>
-        </geometry>
-        <material name="Orange"/>
-      </visual>
-      <collision>
-        <origin xyz="0 0 0" rpy="0 0 0"/>
-        <geometry>
-          <mesh filename="package://iiwa_description/meshes/iiwa14/collision/link_2.stl"/>
+          <mesh filename="package://iiwa_gazebo/meshes/iiwa14/visual/link_2.stl"/>
+        </geometry>
+        <material name="Orange"/>
+      </visual>
+      <collision>
+        <origin xyz="0 0 0" rpy="0 0 0"/>
+        <geometry>
+          <mesh filename="package://iiwa_gazebo/meshes/iiwa14/collision/link_2.stl"/>
         </geometry>
         <material name="Orange"/>
@@ -137,12 +137,12 @@
         <origin xyz="0 0 0" rpy="0 0 0"/>
         <geometry>
-          <mesh filename="package://iiwa_description/meshes/iiwa14/visual/link_3.stl"/>
-        </geometry>
-        <material name="Orange"/>
-      </visual>
-      <collision>
-        <origin xyz="0 0 0" rpy="0 0 0"/>
-        <geometry>
-          <mesh filename="package://iiwa_description/meshes/iiwa14/collision/link_3.stl"/>
+          <mesh filename="package://iiwa_gazebo/meshes/iiwa14/visual/link_3.stl"/>
+        </geometry>
+        <material name="Orange"/>
+      </visual>
+      <collision>
+        <origin xyz="0 0 0" rpy="0 0 0"/>
+        <geometry>
+          <mesh filename="package://iiwa_gazebo/meshes/iiwa14/collision/link_3.stl"/>
         </geometry>
         <material name="Orange"/>
@@ -172,12 +172,12 @@
         <origin xyz="0 0 0" rpy="0 0 0"/>
         <geometry>
-          <mesh filename="package://iiwa_description/meshes/iiwa14/visual/link_4.stl"/>
-        </geometry>
-        <material name="Orange"/>
-      </visual>
-      <collision>
-        <origin xyz="0 0 0" rpy="0 0 0"/>
-        <geometry>
-          <mesh filename="package://iiwa_description/meshes/iiwa14/collision/link_4.stl"/>
+          <mesh filename="package://iiwa_gazebo/meshes/iiwa14/visual/link_4.stl"/>
+        </geometry>
+        <material name="Orange"/>
+      </visual>
+      <collision>
+        <origin xyz="0 0 0" rpy="0 0 0"/>
+        <geometry>
+          <mesh filename="package://iiwa_gazebo/meshes/iiwa14/collision/link_4.stl"/>
         </geometry>
         <material name="Orange"/>
@@ -207,12 +207,12 @@
         <origin xyz="0 0 0" rpy="0 0 0"/>
         <geometry>
-          <mesh filename="package://iiwa_description/meshes/iiwa14/visual/link_5.stl"/>
-        </geometry>
-        <material name="Orange"/>
-      </visual>
-      <collision>
-        <origin xyz="0 0 0" rpy="0 0 0"/>
-        <geometry>
-          <mesh filename="package://iiwa_description/meshes/iiwa14/collision/link_5.stl"/>
+          <mesh filename="package://iiwa_gazebo/meshes/iiwa14/visual/link_5.stl"/>
+        </geometry>
+        <material name="Orange"/>
+      </visual>
+      <collision>
+        <origin xyz="0 0 0" rpy="0 0 0"/>
+        <geometry>
+          <mesh filename="package://iiwa_gazebo/meshes/iiwa14/collision/link_5.stl"/>
         </geometry>
         <material name="Orange"/>
@@ -242,12 +242,12 @@
         <origin xyz="0 0 0" rpy="0 0 0"/>
         <geometry>
-          <mesh filename="package://iiwa_description/meshes/iiwa14/visual/link_6.stl"/>
-        </geometry>
-        <material name="Orange"/>
-      </visual>
-      <collision>
-        <origin xyz="0 0 0" rpy="0 0 0"/>
-        <geometry>
-          <mesh filename="package://iiwa_description/meshes/iiwa14/collision/link_6.stl"/>
+          <mesh filename="package://iiwa_gazebo/meshes/iiwa14/visual/link_6.stl"/>
+        </geometry>
+        <material name="Orange"/>
+      </visual>
+      <collision>
+        <origin xyz="0 0 0" rpy="0 0 0"/>
+        <geometry>
+          <mesh filename="package://iiwa_gazebo/meshes/iiwa14/collision/link_6.stl"/>
         </geometry>
         <material name="Orange"/>
@@ -277,5 +277,5 @@
         <origin xyz="0 0 0" rpy="0 0 0"/>
         <geometry>
-          <mesh filename="package://iiwa_description/meshes/iiwa14/visual/link_7.stl"/>
+          <mesh filename="package://iiwa_gazebo/meshes/iiwa14/visual/link_7.stl"/>
         </geometry>
         <material name="Grey"/>
@@ -284,5 +284,5 @@
         <origin xyz="0 0 0" rpy="0 0 0"/>
         <geometry>
-          <mesh filename="package://iiwa_description/meshes/iiwa14/collision/link_7.stl"/>
+          <mesh filename="package://iiwa_gazebo/meshes/iiwa14/collision/link_7.stl"/>
         </geometry>
         <material name="Grey"/>
