Commit message: Started to implement both controllers: Position + Effort

File: src/iiwa_gazebo/urdf/iiwa.gazebo.xacro (robot description, xacro)
@@ -4,8 +4,12 @@
     <!-- Load Gazebo lib and set the robot namespace -->
     <gazebo>
-	    <plugin name="iiwa_gazebo_plugin" filename="libiiwa_gazebo_plugin.so"/>
+      <plugin name="gazebo_ros_control" filename="libgazebo_ros_control.so">
+        <robotNamespace>/${robot_name}</robotNamespace>
+        <legacyModeNS>true</legacyModeNS>
+      </plugin>
+	  <plugin name="iiwa_gazebo_plugin" filename="libiiwa_gazebo_plugin.so"/>
     </gazebo>
     <!-- Link0 -->
-    <gazebo reference="iiwa_link_0">
+    <gazebo reference="${robot_name}_link_0">
       <material>Gazebo/Grey</material>
       <mu1>0.2</mu1>
@@ -13,5 +17,5 @@
     </gazebo>
     <!-- Link1 -->
-    <gazebo reference="iiwa_link_1">
+    <gazebo reference="${robot_name}_link_1">
       <material>Gazebo/Orange</material>
       <mu1>0.2</mu1>
@@ -22,5 +26,5 @@
     </gazebo>
     <!-- Link2 -->
-    <gazebo reference="iiwa_link_2">
+    <gazebo reference="${robot_name}_link_2">
       <material>Gazebo/Orange</material>
       <mu1>0.2</mu1>
@@ -31,5 +35,5 @@
     </gazebo>
     <!-- Link3 -->
-    <gazebo reference="iiwa_link_3">
+    <gazebo reference="${robot_name}_link_3">
       <material>Gazebo/Orange</material>
       <mu1>0.2</mu1>
@@ -40,5 +44,5 @@
     </gazebo>
     <!-- Link4 -->
-    <gazebo reference="iiwa_link_4">
+    <gazebo reference="${robot_name}_link_4">
       <material>Gazebo/Orange</material>
       <mu1>0.2</mu1>
@@ -49,5 +53,5 @@
     </gazebo>
     <!-- Link5 -->
-    <gazebo reference="iiwa_link_5">
+    <gazebo reference="${robot_name}_link_5">
       <material>Gazebo/Orange</material>
       <mu1>0.2</mu1>
@@ -58,5 +62,5 @@
     </gazebo>
     <!-- Link6 -->
-    <gazebo reference="iiwa_link_6">
+    <gazebo reference="${robot_name}_link_6">
       <material>Gazebo/Orange</material>
       <mu1>0.2</mu1>
@@ -67,5 +71,5 @@
     </gazebo>
     <!-- Link7 -->
-    <gazebo reference="iiwa_link_7">
+    <gazebo reference="${robot_name}_link_7">
       <material>Gazebo/Grey</material>
       <mu1>0.2</mu1>

File: src/iiwa_gazebo/urdf/iiwa14.urdf.xacro (robot description, xacro)
@@ -4,9 +4,10 @@
   <!--Import the lbr iiwa macro -->
   <xacro:include filename="$(find iiwa_gazebo)/urdf/iiwa14.xacro"/>
+  <xacro:arg name="hardware_interface" default="PositionJointInterface"/>
   <xacro:arg name="robot_name" default="iiwa"/>
   <!-- Fix to world just for testing -->
   <link name="world"/>
   <!--iiwa-->
-  <xacro:iiwa14 robot_name="$(arg robot_name)" parent="world">
+  <xacro:iiwa14 hardware_interface="$(arg hardware_interface)" robot_name="$(arg robot_name)" parent="world">
     <origin xyz="0 0 0.0" rpy="0 0 0"/>
   </xacro:iiwa14>

File: src/iiwa_gazebo/urdf/iiwa14.xacro (robot description, xacro)
@@ -2,4 +2,6 @@
   <!-- Import all Gazebo-customization elements, including Gazebo colors -->
   <xacro:include filename="$(find iiwa_gazebo)/urdf/iiwa.gazebo.xacro" />
+  <!-- Import Transmissions -->
+  <xacro:include filename="$(find iiwa_gazebo)/urdf/iiwa.transmission.xacro"/>
   <!-- Include Utilities -->
   <xacro:include filename="$(find iiwa_gazebo)/urdf/utilities.xacro" />
@@ -10,5 +12,5 @@
   <xacro:property name="max_effort" value="300"/>
   <xacro:property name="max_velocity" value="10"/>
-  <xacro:macro name="iiwa14" params="parent robot_name *origin">
+  <xacro:macro name="iiwa14" params="parent hardware_interface robot_name *origin">
     <!--joint between {parent} and link_0-->
     <joint name="${parent}_${robot_name}_joint" type="fixed">
@@ -306,4 +308,5 @@
     <!--Extensions -->
     <xacro:iiwa_gazebo robot_name="${robot_name}" />
+    <xacro:iiwa_transmission hardware_interface="${hardware_interface}"/>
   </xacro:macro>
 </robot>

Commit message: Revert "Started to implement both controllers: Position + Effort"
This reverts commit f9a6d78b6b1228d3c03c82e0c57b3f90eb5e5f37.

File: src/iiwa_gazebo/urdf/iiwa.gazebo.xacro (robot description, xacro)
@@ -4,12 +4,8 @@
     <!-- Load Gazebo lib and set the robot namespace -->
     <gazebo>
-      <plugin name="gazebo_ros_control" filename="libgazebo_ros_control.so">
-        <robotNamespace>/${robot_name}</robotNamespace>
-        <legacyModeNS>true</legacyModeNS>
-      </plugin>
-	  <plugin name="iiwa_gazebo_plugin" filename="libiiwa_gazebo_plugin.so"/>
+	    <plugin name="iiwa_gazebo_plugin" filename="libiiwa_gazebo_plugin.so"/>
     </gazebo>
     <!-- Link0 -->
-    <gazebo reference="${robot_name}_link_0">
+    <gazebo reference="iiwa_link_0">
       <material>Gazebo/Grey</material>
       <mu1>0.2</mu1>
@@ -17,5 +13,5 @@
     </gazebo>
     <!-- Link1 -->
-    <gazebo reference="${robot_name}_link_1">
+    <gazebo reference="iiwa_link_1">
       <material>Gazebo/Orange</material>
       <mu1>0.2</mu1>
@@ -26,5 +22,5 @@
     </gazebo>
     <!-- Link2 -->
-    <gazebo reference="${robot_name}_link_2">
+    <gazebo reference="iiwa_link_2">
       <material>Gazebo/Orange</material>
       <mu1>0.2</mu1>
@@ -35,5 +31,5 @@
     </gazebo>
     <!-- Link3 -->
-    <gazebo reference="${robot_name}_link_3">
+    <gazebo reference="iiwa_link_3">
       <material>Gazebo/Orange</material>
       <mu1>0.2</mu1>
@@ -44,5 +40,5 @@
     </gazebo>
     <!-- Link4 -->
-    <gazebo reference="${robot_name}_link_4">
+    <gazebo reference="iiwa_link_4">
       <material>Gazebo/Orange</material>
       <mu1>0.2</mu1>
@@ -53,5 +49,5 @@
     </gazebo>
     <!-- Link5 -->
-    <gazebo reference="${robot_name}_link_5">
+    <gazebo reference="iiwa_link_5">
       <material>Gazebo/Orange</material>
       <mu1>0.2</mu1>
@@ -62,5 +58,5 @@
     </gazebo>
     <!-- Link6 -->
-    <gazebo reference="${robot_name}_link_6">
+    <gazebo reference="iiwa_link_6">
       <material>Gazebo/Orange</material>
       <mu1>0.2</mu1>
@@ -71,5 +67,5 @@
     </gazebo>
     <!-- Link7 -->
-    <gazebo reference="${robot_name}_link_7">
+    <gazebo reference="iiwa_link_7">
       <material>Gazebo/Grey</material>
       <mu1>0.2</mu1>

File: src/iiwa_gazebo/urdf/iiwa14.urdf.xacro (robot description, xacro)
@@ -4,10 +4,9 @@
   <!--Import the lbr iiwa macro -->
   <xacro:include filename="$(find iiwa_gazebo)/urdf/iiwa14.xacro"/>
-  <xacro:arg name="hardware_interface" default="PositionJointInterface"/>
   <xacro:arg name="robot_name" default="iiwa"/>
   <!-- Fix to world just for testing -->
   <link name="world"/>
   <!--iiwa-->
-  <xacro:iiwa14 hardware_interface="$(arg hardware_interface)" robot_name="$(arg robot_name)" parent="world">
+  <xacro:iiwa14 robot_name="$(arg robot_name)" parent="world">
     <origin xyz="0 0 0.0" rpy="0 0 0"/>
   </xacro:iiwa14>

File: src/iiwa_gazebo/urdf/iiwa14.xacro (robot description, xacro)
@@ -2,6 +2,4 @@
   <!-- Import all Gazebo-customization elements, including Gazebo colors -->
   <xacro:include filename="$(find iiwa_gazebo)/urdf/iiwa.gazebo.xacro" />
-  <!-- Import Transmissions -->
-  <xacro:include filename="$(find iiwa_gazebo)/urdf/iiwa.transmission.xacro"/>
   <!-- Include Utilities -->
   <xacro:include filename="$(find iiwa_gazebo)/urdf/utilities.xacro" />
@@ -12,5 +10,5 @@
   <xacro:property name="max_effort" value="300"/>
   <xacro:property name="max_velocity" value="10"/>
-  <xacro:macro name="iiwa14" params="parent hardware_interface robot_name *origin">
+  <xacro:macro name="iiwa14" params="parent robot_name *origin">
     <!--joint between {parent} and link_0-->
     <joint name="${parent}_${robot_name}_joint" type="fixed">
@@ -308,5 +306,4 @@
     <!--Extensions -->
     <xacro:iiwa_gazebo robot_name="${robot_name}" />
-    <xacro:iiwa_transmission hardware_interface="${hardware_interface}"/>
   </xacro:macro>
 </robot>
